Commit message: lidar sim inicio

File: description/materials.xacro (robot description, xacro)
@@ -11,4 +11,7 @@
         <color rgba="1.0 1.0 1.0 1.0"/>
     </material>
+    <material name="blue">
+        <color rgba="0.0 0.0 1.0 1.0"/>
+    </material>
     <material name="black">
         <color rgba="0.0 0.0 0.0 1.0"/>

File: description/mower_robot.urdf.xacro (robot description, xacro)
@@ -3,3 +3,4 @@
     <xacro:include filename="robot_frame.xacro" />
     <xacro:include filename="ros2_control.xacro" />
+    <xacro:include filename="lidar.xacro" />
 </robot>
