Commit message: lidar simulado terminado

File: description/lidar.xacro (robot description, xacro)
@@ -23,8 +23,8 @@
     <joint name="lidar_joint" type="fixed">
         <parent link="lidar_stick_link"/>
-        <child link="lidar_link"/>
+        <child link="laser_frame"/>
         <origin xyz="0.0 0.0 0.05" rpy="0.0 0.0 0.0"/>
     </joint>
-    <link name="lidar_link">
+    <link name="laser_frame">
         <visual>
             <geometry>
@@ -41,3 +41,27 @@
         <xacro:cylinder_inertia m="0.2" r="0.07" h="0.04"/>
     </link>
+    <gazebo reference="laser_frame">
+        <sensor name='lidar' type='gpu_lidar'>
+            <pose>0 0 0 0 0 0</pose>
+            <topic>scan</topic>
+            <update_rate>10</update_rate>
+            <lidar>
+                <scan>
+                    <horizontal>
+                        <samples>360</samples>
+                        <resolution>1</resolution>
+                        <min_angle>-3.14</min_angle>
+                        <max_angle>3.14</max_angle>
+                    </horizontal>
+                </scan>
+                <range>
+                    <min>0.3</min>
+                    <max>12.0</max>
+                </range>
+            </lidar>
+            <gz_frame_id>laser_frame</gz_frame_id>
+            <always_on>1</always_on>
+            <visualize>false</visualize>
+        </sensor>
+    </gazebo>
 </robot>
