Commit message: casi modelo

File: description/robot_frame.xacro (robot description, xacro)
@@ -1,4 +1,5 @@
 <?xml version="1.0"?>
 <robot xmlns:xacro="http://www.ros.org/wiki/xacro">
+    <!-- COLORS FOR ROBOT VISUALIZATION IN SIMULATION -->
     <material name="red">
         <color rgba="1.0 0.0 0.0 1.0"/>
@@ -13,19 +14,76 @@
         <color rgba="0.0 0.0 0.0 1.0"/>
     </material>
+    <!-- CONSTANT DEFNITIONS -->
+    <xacro:property name="robot_size_x" value="0.5"/>
+    <xacro:property name="robot_size_y" value="0.3"/>
+    <xacro:property name="robot_size_z" value="0.1"/>
+    <xacro:property name="radius_wheel" value="0.1" />
+    <xacro:property name="height_wheel" value="0.05" />
+    <xacro:property name="idler_wheel_radius" value="0.05" />
+    <!-- BASE LINK -->
     <link name="base_link">
     </link>
-    <joint name="robot_join" type="fixed">
+    <!-- ROBOT JOINT (BASE LINK - ROBOT'S FRAME) -->
+    <joint name="robot_joint" type="fixed">
         <parent link="base_link"/>
         <child link="robot_link"/>
-        <origin xyz="-0.1 0.0  0.0"/>
+        <origin xyz="${-radius_wheel} 0.0  0.0"/>
     </joint>
+    <!-- ROBOT LINK (ROBOT'S FRAME) -->
     <link name="robot_link">
         <visual>
-            <origin xyz="0.25 0.0 0.05"/>
+            <origin xyz="${robot_size_x / 2} 0.0 ${robot_size_z / 2}"/>
             <geometry>
-                <box size="0.5 0.3 0.1"/>
+                <box size="${robot_size_x} ${robot_size_y} ${robot_size_z}"/>
             </geometry>
             <material name="red"/>
         </visual>
     </link>
+    <!-- LEFT WHEEL JOINT-->
+    <joint name="left_wheel_joint" type="continuous">
+        <parent link="base_link"/>
+        <child link="left_wheel_link"/>
+        <origin xyz="0.0 ${robot_size_y / 2 + height_wheel / 2} 0.05" rpy="${-pi / 2} 0.0 0.0"/>
+        <axis xyz="0.0 0.0 1.0"/>
+    </joint>
+    <!-- LEFT WHEEL LINK -->
+    <link name="left_wheel_link">
+        <visual>
+            <geometry>
+                <cylinder radius="${radius_wheel}" length="${height_wheel}"/>
+            </geometry>
+            <material name="black"/>
+        </visual>
+    </link>
+    <!-- RIGHT  WHEEL JOINT-->
+    <joint name="right_wheel_joint" type="continuous">
+        <parent link="base_link"/>
+        <child link="right_wheel_link"/>
+        <origin xyz="0.0 ${-robot_size_y / 2 - height_wheel / 2} 0.05" rpy="${pi / 2} 0.0 0.0"/>
+        <axis xyz="0.0 0.0 -1.0"/>
+    </joint>
+    <!-- RIGHT WHEEL LINK -->
+    <link name="right_wheel_link">
+        <visual>
+            <geometry>
+                <cylinder radius="${radius_wheel}" length="${height_wheel}"/>
+            </geometry>
+            <material name="black"/>
+        </visual>
+    </link>
+    <!-- IDLER WHEEL JOINT -->
+    <joint name="idler_wheel_joint" type="fixed">
+        <parent link="robot_link"/>
+        <child link="idler_wheel_link"/>
+        <origin xyz="${robot_size_x - 0.1} 0.0 0.0"/>
+    </joint>
+    <!-- IDLER WHEEL LINK -->
+    <link name="idler_wheel_link">
+        <visual>
+            <geometry>
+                <sphere radius="${idler_wheel_radius}"/>
+            </geometry>
+            <material name="black"/>
+        </visual>
+    </link>
 </robot>

Commit message: urdf file finished

File: description/robot_frame.xacro (robot description, xacro)
@@ -1,24 +1,7 @@
 <?xml version="1.0"?>
 <robot xmlns:xacro="http://www.ros.org/wiki/xacro">
-    <!-- COLORS FOR ROBOT VISUALIZATION IN SIMULATION -->
-    <material name="red">
-        <color rgba="1.0 0.0 0.0 1.0"/>
-    </material>
-    <material name="green">
-        <color rgba="0.0 1.0 0.0 1.0"/>
-    </material>
-    <material name="white">
-        <color rgba="1.0 1.0 1.0 1.0"/>
-    </material>
-    <material name="black">
-        <color rgba="0.0 0.0 0.0 1.0"/>
-    </material>
-    <!-- CONSTANT DEFNITIONS -->
-    <xacro:property name="robot_size_x" value="0.5"/>
-    <xacro:property name="robot_size_y" value="0.3"/>
-    <xacro:property name="robot_size_z" value="0.1"/>
-    <xacro:property name="radius_wheel" value="0.1" />
-    <xacro:property name="height_wheel" value="0.05" />
-    <xacro:property name="idler_wheel_radius" value="0.05" />
+    <xacro:include filename="materials.xacro" />
+    <xacro:include filename="constants.xacro" />
+    <xacro:include filename="inertial_properties.xacro" />
     <!-- BASE LINK -->
     <link name="base_link">
@@ -39,4 +22,11 @@
             <material name="red"/>
         </visual>
+        <collision>
+            <origin xyz="${robot_size_x / 2} 0.0 ${robot_size_z / 2}"/>
+            <geometry>
+                <box size="${robot_size_x} ${robot_size_y} ${robot_size_z}"/>
+            </geometry>
+        </collision>
+        <xacro:box_inertia m="5" w="${robot_size_x}" d="${robot_size_y}" h="${robot_size_z}"/>
     </link>
     <!-- LEFT WHEEL JOINT-->
@@ -55,4 +45,10 @@
             <material name="black"/>
         </visual>
+        <collision>
+            <geometry>
+                <cylinder radius="${radius_wheel}" length="${height_wheel}"/>
+            </geometry>
+        </collision>
+        <xacro:cylinder_inertia m="0.5" r="${radius_wheel}" h="${height_wheel}"/>
     </link>
     <!-- RIGHT  WHEEL JOINT-->
@@ -71,4 +67,11 @@
             <material name="black"/>
         </visual>
+        <collision>
+            <geometry>
+                <cylinder radius="${radius_wheel}" length="${height_wheel}"/>
+            </geometry>
+            <material name="black"/>
+        </collision>
+        <xacro:cylinder_inertia m="0.5" r="${radius_wheel}" h="${height_wheel}"/>
     </link>
     <!-- IDLER WHEEL JOINT -->
@@ -86,4 +89,11 @@
             <material name="black"/>
         </visual>
+        <collision>
+            <geometry>
+                <sphere radius="${idler_wheel_radius}"/>
+            </geometry>
+            <material name="black"/>
+        </collision>
+        <xacro:sphere_inertia m="0.5" r="${idler_wheel_radius}"/>
     </link>
 </robot>

Commit message: robot se mueve bien

File: description/robot_frame.xacro (robot description, xacro)
@@ -28,5 +28,5 @@
             </geometry>
         </collision>
-        <xacro:box_inertia m="5" w="${robot_size_x}" d="${robot_size_y}" h="${robot_size_z}"/>
+        <xacro:box_inertia m="3.5" w="${robot_size_x}" d="${robot_size_y}" h="${robot_size_z}"/>
     </link>
     <!-- LEFT WHEEL JOINT-->
@@ -50,12 +50,12 @@
             </geometry>
         </collision>
-        <xacro:cylinder_inertia m="0.5" r="${radius_wheel}" h="${height_wheel}"/>
+        <xacro:cylinder_inertia m="1.5" r="${radius_wheel}" h="${height_wheel}"/>
     </link>
-    <!-- RIGHT  WHEEL JOINT-->
+    <!-- RIGHT WHEEL JOINT-->
     <joint name="right_wheel_joint" type="continuous">
         <parent link="base_link"/>
         <child link="right_wheel_link"/>
-        <origin xyz="0.0 ${-robot_size_y / 2 - height_wheel / 2} 0.05" rpy="${pi / 2} 0.0 0.0"/>
-        <axis xyz="0.0 0.0 -1.0"/>
+        <origin xyz="0.0 ${-robot_size_y / 2 - height_wheel / 2} 0.05" rpy="${-pi / 2} 0.0 0.0"/>
+        <axis xyz="0.0 0.0 1.0"/>
     </joint>
     <!-- RIGHT WHEEL LINK -->
@@ -73,5 +73,5 @@
             <material name="black"/>
         </collision>
-        <xacro:cylinder_inertia m="0.5" r="${radius_wheel}" h="${height_wheel}"/>
+        <xacro:cylinder_inertia m="1.5" r="${radius_wheel}" h="${height_wheel}"/>
     </link>
     <!-- IDLER WHEEL JOINT -->

Commit message: nav2_casi

File: description/robot_frame.xacro (robot description, xacro)
@@ -7,4 +7,11 @@
     <link name="base_link">
     </link>
+    <!-- BASE FOOTPRINT LINK AND JOIN -->
+    <joint name="base_footprint_joint" type="fixed">
+        <parent link="base_link"/>
+        <child link="base_footprint"/>
+        <origin xyz="0.0 0.0 0.0" rpy="0.0 0.0 0.0"/>
+    </joint>
+    <link name="base_footprint"></link>
     <!-- ROBOT JOINT (BASE LINK - ROBOT'S FRAME) -->
     <joint name="robot_joint" type="fixed">
