Commit message: avance

File: description/constants.xacro (robot description, xacro)
@@ -2,9 +2,9 @@
 <robot xmlns:xacro="http://www.ros.org/wiki/xacro">
     <!-- CONSTANT DEFNITIONS -->
-    <xacro:property name="robot_size_x" value="0.5"/>
-    <xacro:property name="robot_size_y" value="0.3"/>
-    <xacro:property name="robot_size_z" value="0.1"/>
-    <xacro:property name="radius_wheel" value="0.1" />
-    <xacro:property name="height_wheel" value="0.05" />
-    <xacro:property name="idler_wheel_radius" value="0.05" />
+    <xacro:property name="robot_size_x" value="0.22"/>
+    <xacro:property name="robot_size_y" value="0.15"/>
+    <xacro:property name="robot_size_z" value="0.07"/>
+    <xacro:property name="radius_wheel" value="0.033" />
+    <xacro:property name="height_wheel" value="0.026" />
+    <xacro:property name="idler_wheel_radius" value="0.15" />
 </robot>

File: description/lidar.xacro (robot description, xacro)
@@ -19,5 +19,5 @@
             <material name="green"/>
         </collision>
-        <xacro:cylinder_inertia m="0.1" r="0.02" h="0.2"/>
+        <xacro:cylinder_inertia m="0.1" r="0.02" h="0.1"/>
     </link>
     <joint name="lidar_joint" type="fixed">

File: description/robot_frame.xacro (robot description, xacro)
@@ -7,5 +7,5 @@
     <link name="base_link">
     </link>
-    <!-- BASE FOOTPRINT LINK AND JOIN -->
+    <!-- BASE FOOTPRINT LINK AND JOINT -->
     <joint name="base_footprint_joint" type="fixed">
         <parent link="base_link"/>
@@ -35,5 +35,5 @@
             </geometry>
         </collision>
-        <xacro:box_inertia m="3.5" w="${robot_size_x}" d="${robot_size_y}" h="${robot_size_z}"/>
+        <xacro:box_inertia m="2.0" w="${robot_size_x}" d="${robot_size_y}" h="${robot_size_z}"/>
     </link>
     <!-- LEFT WHEEL JOINT-->
@@ -41,5 +41,5 @@
         <parent link="base_link"/>
         <child link="left_wheel_link"/>
-        <origin xyz="0.0 ${robot_size_y / 2 + height_wheel / 2} 0.05" rpy="${-pi / 2} 0.0 0.0"/>
+        <origin xyz="0.0 ${robot_size_y / 2 + height_wheel / 2} ${radius_wheel - idler_wheel_radius}" rpy="${-pi / 2} 0.0 0.0"/>
         <axis xyz="0.0 0.0 1.0"/>
     </joint>
@@ -57,5 +57,5 @@
             </geometry>
         </collision>
-        <xacro:cylinder_inertia m="1.5" r="${radius_wheel}" h="${height_wheel}"/>
+        <xacro:cylinder_inertia m="1.0" r="${radius_wheel}" h="${height_wheel}"/>
     </link>
     <!-- RIGHT WHEEL JOINT-->
@@ -63,5 +63,5 @@
         <parent link="base_link"/>
         <child link="right_wheel_link"/>
-        <origin xyz="0.0 ${-robot_size_y / 2 - height_wheel / 2} 0.05" rpy="${-pi / 2} 0.0 0.0"/>
+        <origin xyz="0.0 ${-robot_size_y / 2 - height_wheel / 2} ${radius_wheel - idler_wheel_radius}" rpy="${-pi / 2} 0.0 0.0"/>
         <axis xyz="0.0 0.0 1.0"/>
     </joint>
@@ -80,5 +80,5 @@
             <material name="black"/>
         </collision>
-        <xacro:cylinder_inertia m="1.5" r="${radius_wheel}" h="${height_wheel}"/>
+        <xacro:cylinder_inertia m="1.0" r="${radius_wheel}" h="${height_wheel}"/>
     </link>
     <!-- IDLER WHEEL JOINT -->

Commit message: urdf adaptado

File: description/constants.xacro (robot description, xacro)
@@ -7,4 +7,4 @@
     <xacro:property name="radius_wheel" value="0.033" />
     <xacro:property name="height_wheel" value="0.026" />
-    <xacro:property name="idler_wheel_radius" value="0.15" />
+    <xacro:property name="idler_wheel_radius" value="0.015" />
 </robot>

File: description/lidar.xacro (robot description, xacro)
@@ -9,5 +9,5 @@
         <visual>
             <geometry>
-                <cylinder radius="0.02" length="0.1"/>
+                <cylinder radius="0.01" length="0.1"/>
             </geometry>
             <material name="green"/>
@@ -15,9 +15,9 @@
         <collision>
             <geometry>
-                <cylinder radius="0.02" length="0.2"/>
+                <cylinder radius="0.01" length="0.1"/>
             </geometry>
             <material name="green"/>
         </collision>
-        <xacro:cylinder_inertia m="0.1" r="0.02" h="0.1"/>
+        <xacro:cylinder_inertia m="0.1" r="0.01" h="0.1"/>
     </link>
     <joint name="lidar_joint" type="fixed">
@@ -29,5 +29,5 @@
         <visual>
             <geometry>
-                <cylinder radius="0.07" length="0.04"/>
+                <cylinder radius="0.035" length="0.02"/>
             </geometry>
             <material name="blue"/>
@@ -35,9 +35,9 @@
         <collision>
             <geometry>
-                <cylinder radius="0.07" length="0.04"/>
+                <cylinder radius="0.035" length="0.02"/>
             </geometry>
             <material name="blue"/>
         </collision>
-        <xacro:cylinder_inertia m="0.2" r="0.07" h="0.04"/>
+        <xacro:cylinder_inertia m="0.2" r="0.035" h="0.02"/>
     </link>
     <gazebo reference="laser_frame">

File: description/robot_frame.xacro (robot description, xacro)
@@ -86,5 +86,5 @@
         <parent link="robot_link"/>
         <child link="idler_wheel_link"/>
-        <origin xyz="${robot_size_x - 0.1} 0.0 0.0"/>
+        <origin xyz="${robot_size_x - 0.05} 0.0 0.0"/>
     </joint>
     <!-- IDLER WHEEL LINK -->
